Commit message: now supports multi-drone configuration

File: libraries/tum_simulator/cvg_sim_gazebo/urdf/quadrotor_sensors.urdf.xacro (robot description, xacro)
@@ -11,5 +11,5 @@
     <!-- Sonar height sensor -->
     <xacro:include filename="$(find cvg_sim_gazebo)/urdf/sensors/sonar_sensor.urdf.xacro" />
-    <xacro:sonar_sensor name="sonar" parent="base_link" ros_topic="sonar_height" update_rate="10" min_range="0.01" max_range="3.0" field_of_view="${40*M_PI/180}" ray_count="3">
+    <xacro:sonar_sensor name="sonar" parent="base_link" ros_topic="$(arg tf_prefix)/sonar_height" update_rate="10" min_range="0.01" max_range="3.0" field_of_view="${40*M_PI/180}" ray_count="3">
       <origin xyz="-0.15 0.0 0.0" rpy="0 ${90*M_PI/180} 0"/>
     </xacro:sonar_sensor>

File: libraries/tum_simulator/cvg_sim_gazebo/urdf/sensors/generic_camera.urdf.xacro (robot description, xacro)
@@ -74,9 +74,9 @@
         </camera>
         <plugin name="${name}_camera_controller" filename="libgazebo_ros_camera.so">
-	  <cameraName>/${sim_name}/${name}</cameraName>
+            <cameraName>${tf_prefix}/${sim_name}/${name}</cameraName>
           <alwaysOn>true</alwaysOn>
           <updateRate>${update_rate}</updateRate>
-          <imageTopicName>/${sim_name}/${name}/image_raw</imageTopicName>
-          <cameraInfoTopicName>/${sim_name}/${name}/camera_info</cameraInfoTopicName>
+          <imageTopicName>${tf_prefix}/${sim_name}/${name}/image_raw</imageTopicName>
+          <cameraInfoTopicName>${tf_prefix}/${sim_name}/${name}/camera_info</cameraInfoTopicName>
 		  <frameName>${tf_prefix}/ardrone_base_${name}cam</frameName>
         </plugin>

File: libraries/tum_simulator/cvg_sim_gazebo_plugins/urdf/quadrotor_sensors.urdf.xacro (robot description, xacro)
@@ -14,6 +14,7 @@
         <updateRate>100.0</updateRate>
         <bodyName>base_link</bodyName>
-        <frameId>ardrone_base_link</frameId>
-        <topicName>/ardrone/imu</topicName>
+        <!-- TODO : update bodyName?? -->
+        <frameId>$(arg tf_prefix)/base_link</frameId>
+        <topicName>$(arg tf_prefix)/imu</topicName>
         <rpyOffsets>0 0 0</rpyOffsets> <!-- deprecated -->
         <gaussianNoise>0</gaussianNoise>  <!-- deprecated -->
@@ -29,6 +30,6 @@
         <updateRate>10.0</updateRate>
         <bodyName>base_link</bodyName>
-        <topicName>pressure_height</topicName>
-        <altimeterTopicName>altimeter</altimeterTopicName>
+        <topicName>$(arg tf_prefix)/pressure_height</topicName>
+        <altimeterTopicName>$(arg tf_prefix)/altimeter</altimeterTopicName>
         <offset>0</offset>
         <drift>0.1</drift>
@@ -39,5 +40,5 @@
         <updateRate>10.0</updateRate>
         <bodyName>base_link</bodyName>
-        <topicName>magnetic</topicName>
+        <topicName>$(arg tf_prefix)/magnetic</topicName>
         <offset>0 0 0</offset>
         <drift>0.0 0.0 0.0</drift>
@@ -48,6 +49,6 @@
         <updateRate>4.0</updateRate>
         <bodyName>base_link</bodyName>
-        <topicName>fix</topicName>
-        <velocityTopicName>fix_velocity</velocityTopicName>
+        <topicName>$(arg tf_prefix)/fix</topicName>
+        <velocityTopicName>$(arg tf_prefix)/fix_velocity</velocityTopicName>
         <drift>5.0 5.0 5.0</drift>
         <gaussianNoise>0.1 0.1 0.1</gaussianNoise>
@@ -59,5 +60,5 @@
         <updateRate>100.0</updateRate>
         <bodyName>base_link</bodyName>
-		<topicName>ground_truth/state</topicName>
+        <topicName>$(arg tf_prefix)/ground_truth/state</topicName>
         <gaussianNoise>0.0</gaussianNoise>
         <frameName>map</frameName>

File: libraries/tum_simulator/cvg_sim_gazebo_plugins/urdf/quadrotor_simple_controller.urdf.xacro (robot description, xacro)
@@ -1,44 +1,47 @@
 <?xml version="1.0"?>
 <robot
-xmlns:controller="http://playerstage.sourceforge.net/gazebo/xmlschema/#controller"
-xmlns:xacro="http://ros.org/wiki/xacro"
->
-  <!-- Quadrotor Simple Controller Plugin -->
-  <xacro:macro name="quadrotor_controller">
-    <gazebo>
-      <plugin name="quadrotor_simple_controller" filename="libhector_gazebo_quadrotor_simple_controller.so">
-        <alwaysOn>true</alwaysOn>
-        <updateRate>0.0</updateRate>
-        <bodyName>base_link</bodyName>
-        <stateTopic>ground_truth/state</stateTopic>
-        <imuTopic>ardrone/imu</imuTopic>
-        <topicName>cmd_vel</topicName>
-        <rollpitchProportionalGain>10.0</rollpitchProportionalGain>
-        <rollpitchDifferentialGain>5.0</rollpitchDifferentialGain>
-        <rollpitchLimit>0.5</rollpitchLimit>
-        <yawProportionalGain>2.0</yawProportionalGain>
-        <yawDifferentialGain>1.0</yawDifferentialGain>
-        <yawLimit>1.5</yawLimit>
-        <velocityXYProportionalGain>5.0</velocityXYProportionalGain>
-        <velocityXYDifferentialGain>1.0</velocityXYDifferentialGain>
-        <velocityXYLimit>2</velocityXYLimit>
-        <velocityZProportionalGain>5.0</velocityZProportionalGain>
-        <velocityZDifferentialGain>1.0</velocityZDifferentialGain>
-        <velocityZLimit>0.5</velocityZLimit>
-        <maxForce>30</maxForce>
-        <motionSmallNoise>0.05</motionSmallNoise>
-        <motionDriftNoise>0.03</motionDriftNoise>
-        <motionDriftNoiseTime>5.0</motionDriftNoiseTime>
-      </plugin>
-      <plugin name="quadrotor_state_controller" filename="libhector_gazebo_quadrotor_state_controller.so">
-        <alwaysOn>true</alwaysOn>
-        <updateRate>0.0</updateRate>
-        <bodyName>base_link</bodyName>
-        <stateTopic>ground_truth/state</stateTopic>
-        <imuTopic>ardrone/imu</imuTopic>
-        <sonarTopic>sonar_height</sonarTopic>
-        <topicName>cmd_vel</topicName>
-      </plugin>
-    </gazebo>
-  </xacro:macro>
+    xmlns:controller="http://playerstage.sourceforge.net/gazebo/xmlschema/#controller"
+    xmlns:xacro="http://ros.org/wiki/xacro"
+    >
+    <!-- Quadrotor Simple Controller Plugin -->
+    <xacro:macro name="quadrotor_controller">
+        <gazebo>
+            <plugin name="quadrotor_simple_controller" filename="libhector_gazebo_quadrotor_simple_controller.so">
+                <robotNamespace>$(arg tf_prefix)</robotNamespace>
+                <alwaysOn>true</alwaysOn>
+                <updateRate>0.0</updateRate>
+                <bodyName>base_link</bodyName>
+                <stateTopic>ground_truth/state</stateTopic>
+                <imuTopic>imu</imuTopic>
+                <topicName>cmd_vel</topicName>
+                <rollpitchProportionalGain>10.0</rollpitchProportionalGain>
+                <rollpitchDifferentialGain>5.0</rollpitchDifferentialGain>
+                <rollpitchLimit>0.5</rollpitchLimit>
+                <yawProportionalGain>2.0</yawProportionalGain>
+                <yawDifferentialGain>1.0</yawDifferentialGain>
+                <yawLimit>1.5</yawLimit>
+                <velocityXYProportionalGain>5.0</velocityXYProportionalGain>
+                <velocityXYDifferentialGain>1.0</velocityXYDifferentialGain>
+                <velocityXYLimit>2</velocityXYLimit>
+                <velocityZProportionalGain>5.0</velocityZProportionalGain>
+                <velocityZDifferentialGain>1.0</velocityZDifferentialGain>
+                <velocityZLimit>0.5</velocityZLimit>
+                <maxForce>30</maxForce>
+                <motionSmallNoise>0.05</motionSmallNoise>
+                <motionDriftNoise>0.03</motionDriftNoise>
+                <motionDriftNoiseTime>5.0</motionDriftNoiseTime>
+            </plugin>
+            <plugin name="quadrotor_state_controller" filename="libhector_gazebo_quadrotor_state_controller.so">
+                <robotNamespace>$(arg tf_prefix)</robotNamespace>
+                <alwaysOn>true</alwaysOn>
+                <updateRate>0.0</updateRate>
+                <bodyName>base_link</bodyName>
+                <stateTopic>ground_truth/state</stateTopic>
+                <imuTopic>imu</imuTopic>
+                <sonarTopic>sonar_height</sonarTopic>
+                <topicName>cmd_vel</topicName>
+                <navdataTopic>ardrone/navdata</navdataTopic>
+            </plugin>
+        </gazebo>
+    </xacro:macro>
 </robot>
