Commit message: fixed camera topics namespaces issue

File: libraries/tum_simulator/cvg_sim_gazebo/urdf/sensors/generic_camera.urdf.xacro (robot description, xacro)
@@ -1,88 +1,88 @@
 <?xml version="1.0"?>
 <robot xmlns:sensor="http://playerstage.sourceforge.net/gazebo/xmlschema/#sensor"
-xmlns:controller="http://playerstage.sourceforge.net/gazebo/xmlschema/#controller"
-xmlns:xacro="http://ros.org/wiki/xacro">
+    xmlns:controller="http://playerstage.sourceforge.net/gazebo/xmlschema/#controller"
+    xmlns:xacro="http://ros.org/wiki/xacro">
     <xacro:property name="M_PI" value="3.1415926535897931" />
     <xacro:macro name="generic_camera" params="name sim_name parent *origin update_rate res_x res_y image_format hfov tf_prefix:=''">
-      <joint name="${name}_joint" type="fixed">
-        <xacro:insert_block name="origin" />
-        <parent link="${parent}"/>
-        <child link="${name}_link"/>
-      </joint>
-      <link name="${name}_link">
-        <inertial>
-          <mass value="0.001" />
-          <origin xyz="0 0 0" rpy="0 0 0" />
-          <inertia ixx="0.0001" ixy="0" ixz="0" iyy="0.0001" iyz="0" izz="0.0001" />
-        </inertial>
-        <visual>
-          <origin xyz="0 0 0" rpy="0 0 0" />
-          <geometry>
-            <box size="0.01 0.01 0.01" />
-          </geometry>
-	  <material name="Blue">
-      <color rgba="0.0 0.0 0.8 1"/>
-    </material>
-        </visual>
-        <collision>
-          <origin xyz="0 0 0" rpy="0 0 0" />
-          <geometry>
-            <box size="0.01 0.01 0.01" />
-          </geometry>
-        </collision>
-      </link>
-    <joint name="${name}_optical_joint" type="fixed">
-      <origin xyz="0 0 0" rpy="${-M_PI/2} 0.0 ${-M_PI/2}" />
-      <parent link="${name}_link" />
-      <child link="ardrone_base_${name}cam"/>
-    </joint>
-    <link name="ardrone_base_${name}cam">
-      <inertial>
-        <mass value="0.01" />
-        <origin xyz="0 0 0" />
-        <inertia ixx="0.001"  ixy="0.0"  ixz="0.0"
-                 iyy="0.001"  iyz="0.0"
-                 izz="0.001" />
-      </inertial>
-      <visual>
-        <origin xyz="0 0 0" rpy="0 0 0"/>
-        <geometry>
-          <box size="0.001 0.001 0.001" />
-        </geometry>
-      </visual>
-      <collision>
-        <origin xyz="0 0 0" rpy="0 0 0"/>
-        <geometry>
-          <box size="0.001 0.001 0.001" />
-        </geometry>
-      </collision>
-    </link>
-    <gazebo reference="${name}_link">
-      <sensor type="camera" name="${name}_camera_sensor">
-        <update_rate>${update_rate}</update_rate>
-        <camera name="head">
-          <horizontal_fov>${hfov}</horizontal_fov>
-          <image>
-            <width>${res_x}</width>
-            <height>${res_y}</height>
-            <format>${image_format}</format>
-          </image>
-          <clip>0.01
-	    <near>0.01</near>
-            <far>100</far>
-          </clip>
-        </camera>
-        <plugin name="${name}_camera_controller" filename="libgazebo_ros_camera.so">
-            <cameraName>${tf_prefix}/${sim_name}/${name}</cameraName>
-          <alwaysOn>true</alwaysOn>
-          <updateRate>${update_rate}</updateRate>
-          <imageTopicName>${tf_prefix}/${sim_name}/${name}/image_raw</imageTopicName>
-          <cameraInfoTopicName>${tf_prefix}/${sim_name}/${name}/camera_info</cameraInfoTopicName>
-		  <frameName>${tf_prefix}/ardrone_base_${name}cam</frameName>
-        </plugin>
-      </sensor>
-      <turnGravityOff>true</turnGravityOff>
-      <material>PR2/Blue</material>
-    </gazebo>
+        <joint name="${name}_joint" type="fixed">
+            <xacro:insert_block name="origin" />
+            <parent link="${parent}"/>
+            <child link="${name}_link"/>
+        </joint>
+        <link name="${name}_link">
+            <inertial>
+                <mass value="0.001" />
+                <origin xyz="0 0 0" rpy="0 0 0" />
+                <inertia ixx="0.0001" ixy="0" ixz="0" iyy="0.0001" iyz="0" izz="0.0001" />
+            </inertial>
+            <visual>
+                <origin xyz="0 0 0" rpy="0 0 0" />
+                <geometry>
+                    <box size="0.01 0.01 0.01" />
+                </geometry>
+                <material name="Blue">
+                    <color rgba="0.0 0.0 0.8 1"/>
+                </material>
+            </visual>
+            <collision>
+                <origin xyz="0 0 0" rpy="0 0 0" />
+                <geometry>
+                    <box size="0.01 0.01 0.01" />
+                </geometry>
+            </collision>
+        </link>
+        <joint name="${name}_optical_joint" type="fixed">
+            <origin xyz="0 0 0" rpy="${-M_PI/2} 0.0 ${-M_PI/2}" />
+            <parent link="${name}_link" />
+            <child link="ardrone_base_${name}cam"/>
+        </joint>
+        <link name="ardrone_base_${name}cam">
+            <inertial>
+                <mass value="0.01" />
+                <origin xyz="0 0 0" />
+                <inertia ixx="0.001"  ixy="0.0"  ixz="0.0"
+                    iyy="0.001"  iyz="0.0"
+                    izz="0.001" />
+            </inertial>
+            <visual>
+                <origin xyz="0 0 0" rpy="0 0 0"/>
+                <geometry>
+                    <box size="0.001 0.001 0.001" />
+                </geometry>
+            </visual>
+            <collision>
+                <origin xyz="0 0 0" rpy="0 0 0"/>
+                <geometry>
+                    <box size="0.001 0.001 0.001" />
+                </geometry>
+            </collision>
+        </link>
+        <gazebo reference="${name}_link">
+            <sensor type="camera" name="${name}_camera_sensor">
+                <update_rate>${update_rate}</update_rate>
+                <camera name="head">
+                    <horizontal_fov>${hfov}</horizontal_fov>
+                    <image>
+                        <width>${res_x}</width>
+                        <height>${res_y}</height>
+                        <format>${image_format}</format>
+                    </image>
+                    <clip>0.01
+                        <near>0.01</near>
+                        <far>100</far>
+                    </clip>
+                </camera>
+                <plugin name="${name}_camera_controller" filename="libgazebo_ros_camera.so">
+                    <cameraName>${tf_prefix}/${sim_name}/${name}</cameraName>
+                    <alwaysOn>true</alwaysOn>
+                    <updateRate>${update_rate}</updateRate>
+                    <imageTopicName>image_raw</imageTopicName>
+                    <cameraInfoTopicName>camera_info</cameraInfoTopicName>
+                    <frameName>${tf_prefix}/ardrone_base_${name}cam</frameName>
+                </plugin>
+            </sensor>
+            <turnGravityOff>true</turnGravityOff>
+            <material>PR2/Blue</material>
+        </gazebo>
     </xacro:macro>
-  </robot>
+</robot>
